File: PCB/KiCAD-fresh/MagicWiFi/MagicWiFi.kicad_sch (KiCad schematic)
At the start: 6 parts

Commit message: Added basic layout
Parts:
- added U1: ~, MagicWiFi:Barrel_Conn, symbol MagicWiFi:Barrel_Connector
- added U2, U3: ~, MagicWiFi:SMA_EDGELAUNCH, symbol MagicWiFi:Antenna
- added X1, X2: Osc, MagicWiFi:TCXO, symbol MagicWiFi:TCXO
- added X3: Osc, MagicWiFi:Xosc, symbol MagicWiFi:CrystalOsc
Connections:
- net 3v3: now also U1.1 (Inner1)
- net GND: now also U1.2 (Outer)
Changed lines of the file:
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@@
+    (stroke (width 0) (type default))
+  )
+  (wire (pts (xy 41.91 36.83) (xy 46.99 36.83))
     (stroke (width 0) (type default))
   )
@@
     (stroke (width 0) (type default))
   )
+  (wire (pts (xy 68.58 36.83) (xy 72.39 36.83))
+    (stroke (width 0) (type default))
+  )
   (wire (pts (xy 361.95 133.35) (xy 364.49 133.35))
     (stroke (width 0) (type default))
@@
     (effects (font (size 1.27 1.27)) (justify left bottom))
   )
+  (label "3v3" (at 72.39 36.83 0) (fields_autoplaced)
+    (effects (font (size 1.27 1.27)) (justify left bottom))
+  )
   (label "GND" (at 415.29 151.13 0) (fields_autoplaced)
     (effects (font (size 1.27 1.27)) (justify left bottom))
@@
     (effects (font (size 1.27 1.27)) (justify left bottom))
   )
+  (label "GND" (at 41.91 36.83 0) (fields_autoplaced)
+    (effects (font (size 1.27 1.27)) (justify left bottom))
+  )
   (label "3v3" (at 415.29 168.91 0) (fields_autoplaced)
     (effects (font (size 1.27 1.27)) (justify left bottom))
@@
   (label "GND" (at -300.99 151.13 0) (fields_autoplaced)
     (effects (font (size 1.27 1.27)) (justify left bottom))
+  )
+  (symbol (lib_id "MagicWiFi:CrystalOsc") (at 149.86 25.4 0) (unit 1)
+    (in_bom yes) (on_board yes) (dnp no) (fields_autoplaced)
+    (property "Reference" "X3" (at 150.495 12.7 0)
+      (effects (font (size 1.27 1.27)))
+    )
+    (property "Value" "Osc" (at 150.495 15.24 0)
+      (effects (font (size 1.27 1.27)))
+    )
+    (property "Footprint" "MagicWiFi:Xosc" (at 133.35 10.16 0)
+      (effects (font (size 1.27 1.27)) hide)
+    )
+    (property "Datasheet" "https://media.digikey.com/pdf/Data%20Sheets/Jauch%20Quartz%20PDFs/J49SMH_Type_DS.pdf" (at 100.33 12.7 0)
+      (effects (font (size 1.27 1.27)) hide)
+    )
+    (pin "1")
+    (pin "2")
+    (instances
+      (project "MagicWiFi"
+        (path "/aca77577-6dae-43b4-a2d5-29c97c082072"
+          (reference "X3") (unit 1)
+        )
+      )
+    )
   )
   (symbol (lib_id "MagicWiFi:SX1272IMLTRT") (at 364.49 133.35 0) (unit 1)
@@
     )
   )
+  (symbol (lib_id "MagicWiFi:Barrel_Connector") (at 59.69 36.83 0) (unit 1)
+    (in_bom yes) (on_board yes) (dnp no) (fields_autoplaced)
+    (property "Reference" "U1" (at 59.055 25.4 0)
+      (effects (font (size 1.27 1.27)))
+    )
+    (property "Value" "~" (at 59.69 36.83 0)
+      (effects (font (size 1.27 1.27)))
+    )
+    (property "Footprint" "MagicWiFi:Barrel_Conn" (at 39.37 25.4 0)
+      (effects (font (size 1.27 1.27)) hide)
+    )
+    (property "Datasheet" "" (at 59.69 36.83 0)
+      (effects (font (size 1.27 1.27)) hide)
+    )
+    (pin "1")
+    (pin "2")
+    (instances
+      (project "MagicWiFi"
+        (path "/aca77577-6dae-43b4-a2d5-29c97c082072"
+          (reference "U1") (unit 1)
+        )
+      )
+    )
+  )
+  (symbol (lib_id "MagicWiFi:TCXO") (at 337.82 146.05 0) (unit 1)
+    (in_bom yes) (on_board yes) (dnp no) (fields_autoplaced)
+    (property "Reference" "X1" (at 337.82 135.89 0)
+      (effects (font (size 1.27 1.27)))
+    )
+    (property "Value" "Osc" (at 337.82 138.43 0)
+      (effects (font (size 1.27 1.27)))
+    )
+    (property "Footprint" "MagicWiFi:TCXO" (at 322.58 133.35 0)
+      (effects (font (size 1.27 1.27)) hide)
+    )
+    (property "Datasheet" "https://www.jauch.com/downloadfile/57ff7db813438_346edabf994d823423fb/jt32c_180424.pdf" (at 285.75 135.89 0)
+      (effects (font (size 1.27 1.27)) hide)
+    )
+    (pin "1")
+    (pin "3")
+    (pin "3")
+    (pin "4")
+    (instances
+      (project "MagicWiFi"
+        (path "/aca77577-6dae-43b4-a2d5-29c97c082072"
+          (reference "X1") (unit 1)
+        )
+      )
+    )
+  )
   (symbol (lib_id "MagicWiFi:SX1272IMLTRT") (at 363.22 41.91 0) (unit 1)
     (in_bom yes) (on_board yes) (dnp no)
@@
         )
       )
+    )
+  )
+  (symbol (lib_id "MagicWiFi:Antenna") (at 633.73 43.18 180) (unit 1)
+    (in_bom yes) (on_board yes) (dnp no) (fields_autoplaced)
+    (property "Reference" "U3" (at 640.08 43.815 0)
+      (effects (font (size 1.27 1.27)) (justify right))
+    )
+    (property "Value" "~" (at 633.73 43.18 0)
+      (effects (font (size 1.27 1.27)))
+    )
+    (property "Footprint" "MagicWiFi:SMA_EDGELAUNCH" (at 652.78 52.07 0)
+      (effects (font (size 1.27 1.27)) hide)
+    )
+    (property "Datasheet" "" (at 684.53 53.34 0)
+      (effects (font (size 1.27 1.27)) hide)
+    )
+    (pin "1")
+    (pin "2")
+    (pin "3")
+    (pin "4")
+    (pin "5")
+    (instances
+      (project "MagicWiFi"
+        (path "/aca77577-6dae-43b4-a2d5-29c97c082072"
+          (reference "U3") (unit 1)
+        )
+      )
+    )
+  )
+  (symbol (lib_id "MagicWiFi:Antenna") (at 631.19 147.32 180) (unit 1)
+    (in_bom yes) (on_board yes) (dnp no) (fields_autoplaced)
+    (property "Reference" "U2" (at 637.54 147.955 0)
+      (effects (font (size 1.27 1.27)) (justify right))
+    )
+    (property "Value" "~" (at 631.19 147.32 0)
+      (effects (font (size 1.27 1.27)))
+    )
+    (property "Footprint" "MagicWiFi:SMA_EDGELAUNCH" (at 650.24 156.21 0)
+      (effects (font (size 1.27 1.27)) hide)
+    )
+    (property "Datasheet" "" (at 681.99 157.48 0)
+      (effects (font (size 1.27 1.27)) hide)
+    )
+    (pin "1")
+    (pin "2")
+    (pin "3")
+    (pin "4")
+    (pin "5")
+    (instances
+      (project "MagicWiFi"
+        (path "/aca77577-6dae-43b4-a2d5-29c97c082072"
+          (reference "U2") (unit 1)
+        )
+      )
+    )
+  )
+  (symbol (lib_id "MagicWiFi:TCXO") (at 337.82 55.88 0) (unit 1)
+    (in_bom yes) (on_board yes) (dnp no) (fields_autoplaced)
+    (property "Reference" "X2" (at 337.82 45.72 0)
+      (effects (font (size 1.27 1.27)))
+    )
+    (property "Value" "Osc" (at 337.82 48.26 0)
+      (effects (font (size 1.27 1.27)))
+    )
+    (property "Footprint" "MagicWiFi:TCXO" (at 322.58 43.18 0)
+      (effects (font (size 1.27 1.27)) hide)
+    )
+    (property "Datasheet" "https://www.jauch.com/downloadfile/57ff7db813438_346edabf994d823423fb/jt32c_180424.pdf" (at 285.75 45.72 0)
+      (effects (font (size 1.27 1.27)) hide)
+    )
+    (pin "1")
+    (pin "3")
+    (pin "3")
+    (pin "4")
+    (instances
+      (project "MagicWiFi"
+        (path "/aca77577-6dae-43b4-a2d5-29c97c082072"
+          (reference "X2") (unit 1)
+        )
+      )

Commit message: part way through PCB design
Parts:
- removed X3: Osc, MagicWiFi:Xosc, symbol MagicWiFi:CrystalOsc
- added C1: 10uF, Resistor_SMD:R_0805_2012Metric_Pad1.20x1.40mm_HandSolder, symbol Device:C_Small
- added C10, C4, C5, C6, C7, C8, C9: 0.1 uF, Capacitor_SMD:C_0805_2012Metric, symbol Device:C_Small
- added C11, C12: 0.1 nF, Resistor_SMD:R_0805_2012Metric_Pad1.20x1.40mm_HandSolder, symbol Device:C_Small
- added C2: 180 pF, Capacitor_SMD:C_0805_2012Metric, symbol Device:C_Small
- added C3: 14 pF, Capacitor_SMD:C_0805_2012Metric, symbol Device:C_Small
- added FB1: 80 mA min, Resistor_SMD:R_0805_2012Metric_Pad1.20x1.40mm_HandSolder, symbol Device:FerriteBead_Small
- added J1: 702461402, CON_702461402_MOL, symbol MagicWiFi:702461402
- added R1, R2: 60, Resistor_SMD:R_0805_2012Metric_Pad1.20x1.40mm_HandSolder, symbol Device:R_Small
- added R10, R9: 75 Ohm, Resistor_SMD:R_0805_2012Metric_Pad1.20x1.40mm_HandSolder, symbol Device:R_Small
- added R3: 2.32k 1%, Resistor_SMD:R_0805_2012Metric_Pad1.20x1.40mm_HandSolder, symbol Device:R_Small
- added R4: 47k, Resistor_SMD:R_0805_2012Metric_Pad1.20x1.40mm_HandSolder, symbol Device:R_Small
- added R5, R6, R7, R8: 49.9 Ohm, Capacitor_SMD:C_0805_2012Metric, symbol Device:R_Small
- added SW1: SPST-NC, MagicWiFi:KSR223GNCLFG, symbol Switch:SW_Push_Open
- added X0: Osc, MagicWiFi:Xosc, symbol MagicWiFi:CrystalOsc
- added X3: Osc, MagicWiFi:TCXO, symbol MagicWiFi:TCXO
- renumbered U2 to AN1, U3 to AN2, U1 to BATT1
Connections:
- net 3v3: now also X1.4 (Vdc), X2.4 (Vdc), C5.1, C6.1, C7.1, FB1.1, R1.2, R2.2, SW1.2 (B), X3.4 (Vdc)
- net GND: now also X1.3 (Osc), X2.3 (Osc), C1.2, C10.1, C11.1, C12.1, C2.2, C3.1, C4.1, C5.2, C6.2, C7.2, C8.1, C8.2, C9.1, C9.2, J1.9, R3.2, X3.3 (Osc)
- net at MSP430.9 (RST_NMI_SBWTDIO_N): now also R4.1
- net VC2ETH_N: now reaches ARJ1.1 (VC2-)
- net VC2ETH_N: now also R9.2
- net TD_P: now reaches ARJ1.10 (TD+)
- net TD_P: now also ENC1.17 (TPOUT+), R5.1
- net at ARJ1.11 (LEDG+): now also R2.1
- net LEDGN: now reaches ARJ1.12 (LEDG-)
- net LEDGN: now also ENC1.27 (LEDA)
- net at ARJ1.13 (LEDY+): now also R1.1
- net LEDYN: now reaches ARJ1.14 (LEDY-)
- net LEDYN: now also ENC1.26 (LEDB)
- net RD_N: now reaches ARJ1.3 (RD-)
- net RD_N: now also ENC1.12 (TPIN-), R7.2
- net RD_P: now reaches ARJ1.5 (RD+)
- net RD_P: now also ENC1.13 (TPIN+), R8.1
- net VC2ETH_P: now reaches ARJ1.6 (VC2+)
- net VC2ETH_P: now also R10.2
- net TD_N: now reaches ARJ1.8 (TD-)
- net TD_N: now also ENC1.16 (TPOUT-), R6.2
- net TD_C: now reaches ARJ1.9 (TCT)
- net TD_C: now also C4.2, FB1.2, R5.2, R6.1
- net at ENC1.1 (VCAP): now also C1.1
- net ~ETH_RST: now reaches ENC1.10 (~{RESET})
- net at ENC1.14 (RBIAS): now also R3.1
- net OSC1_ETH: now reaches ENC1.23 (OSC1)
- net OSC1_ETH: now also X3.3 (Osc)
- net ~ETH_IRQ: now reaches ENC1.4 (~{INT})
- net ETH_MISO: now reaches ENC1.6 (SO)
- net ETH_MISO: now also J1.3
- net ETH_MOSI: now reaches ENC1.7 (SI)
- net ETH_MOSI: now also J1.1
- net ETH_CLK: now reaches ENC1.8 (SCK)
- net ETH_CLK: now also J1.5
- net ~ETH_CHIPSEL: now reaches ENC1.9 (~{CS})
- net ~ETH_CHIPSEL: now also J1.7
- new net: C10.2, R7.1, R8.2
- new net: C12.2, R10.1
- new net: C3.2, X0.1 (osc1)
- new net: C11.2, R9.1
- new net: C2.1, X0.2 (osc2)
- new net: R4.2, SW1.1 (A)
- new net MSP_TEST: J1.8
- new net MSP_VCC: J1.2
- new net MSP_VCC_TAR: J1.4
- new net ~MSP_RST: J1.10
- no-connect marks 0 -> 11

Commit message: Antenna Design Remade, stolen shamelessly from Sample design by SemTech (Mfgr), other traces routed and Documentation refreshed for components
Parts:
- removed C2: 180 pF, Capacitor_SMD:C_0805_2012Metric, symbol Device:C_Small
- removed C3: 14 pF, Capacitor_SMD:C_0805_2012Metric, symbol Device:C_Small
- removed X0: Osc, MagicWiFi:Xosc, symbol MagicWiFi:CrystalOsc
- added C13, C22: 3.3 pF, Capacitor_SMD:C_0402_1005Metric_Pad0.74x0.62mm_HandSolder, symbol Device:C_Small
- added C14, C15, C17, C23: 47 pF, Capacitor_SMD:C_0402_1005Metric_Pad0.74x0.62mm_HandSolder, symbol Device:C_Small
- added C16: 10 nF, Capacitor_SMD:C_0402_1005Metric_Pad0.74x0.62mm_HandSolder, symbol Device:C_Small
- added C18, C20: 8.2 pF, Capacitor_SMD:C_0402_1005Metric_Pad0.74x0.62mm_HandSolder, symbol Device:C_Small
- added C19: 22 pF, Capacitor_SMD:C_0402_1005Metric_Pad0.74x0.62mm_HandSolder, symbol Device:C_Small
- added C21: 1.5 pF, Capacitor_SMD:C_0402_1005Metric_Pad0.74x0.62mm_HandSolder, symbol Device:C_Small
- added F1: Polyfuse, MagicWiFi:Fuse_BelFuse_0ZCJ0_1206_Metric_3216, symbol Device:Polyfuse
- added L1: 10 nH, Capacitor_SMD:C_0402_1005Metric_Pad0.74x0.62mm_HandSolder, symbol Device:L_Small
- added L2: 33 nH, Inductor_SMD:L_0402_1005Metric_Pad0.77x0.64mm_HandSolder, symbol Device:L_Small
- added L3: 2.7 nH, Inductor_SMD:L_0402_1005Metric_Pad0.77x0.64mm_HandSolder, symbol Device:L_Small
- added L4, L5: 5.6 nH, Inductor_SMD:L_0402_1005Metric_Pad0.77x0.64mm_HandSolder, symbol Device:L_Small
- added R11: 0R, Resistor_SMD:R_0603_1608Metric_Pad0.98x0.95mm_HandSolder, symbol Device:R_Small
- added R12, R13: 0R, Resistor_SMD:R_0402_1005Metric_Pad0.72x0.64mm_HandSolder, symbol Device:R_Small
- J1: MPN (none) -> 702461402
- U1: renamed from MSP430; value MSP430FR2355TDBTR -> MSP430; MPN (none) -> MSP430FR2355TDBTR
- U2: renamed from ARJ1; value ARJM11C7-114-BA-EW2 -> ARJ1; MPN (none) -> ARJM11C7-114-BA-EW2
- U3: renamed from ENC1; value ENC28J60x-SO -> ENC; MPN (none) -> ENC28J60x-SO
- U4: renamed from ATC1; value ATWINC1500-MR210PB1952-T -> ATC; MPN (none) -> ATWINC1500-MR210PB1952-T
- U5: renamed from LoRa1; value SX1272IMLTRT -> LoRa1; MPN (none) -> SX1272IMLTRT
- U6: renamed from LoRa2; value SX1272IMLTRT -> LoRa2; MPN (none) -> SX1272IMLTRT
- X1, X2: MPN (none) -> O 32,0-JT32C-A-K-3,3-LF
- X3: MPN (none) -> O 25,0-JT32C-A-K-3,3-LF
- renumbered BATT1 to BT1
Connections:
- net 3v3: no longer BT1.1 (Inner1), C5.1, C6.1, C7.1, FB1.1, R1.2, R2.2, SW1.2 (B), U1.10 (DVCC), U3.15 (VDDTX), U3.19 (VDDRX), U3.20 (VDDPLL), U3.25 (VDDOSC), U3.28 (VDD), U4.20 (VBAT), U4.23 (VDDIO), U5.1 (VBAT1), U5.15 (VBAT2), U6.1 (VBAT1), U6.15 (VBAT2), X1.4 (Vdc), X2.4 (Vdc)
- net GND: now also AN1.2 (GND), AN1.3 (GND), AN1.4 (GND), AN1.5 (GND), AN2.2 (GND), AN2.3 (GND), AN2.4 (GND), AN2.5 (GND), X1.2 (GND), X2.2 (GND), X3.2 (GND), C13.2, C16.2, C17.2, C18.2, C20.2, C22.2; no longer C8.2, C9.1, X1.3 (Osc), X2.3 (Osc), X3.3 (Osc)
- net at U6.27 (PA_BOOST): now also L3.1
- net at U6.28 (VR_PA): now also C16.1, C17.1, L2.1
- net at U6.4 (XTA): now also X1.3 (Osc)
- net at U5.25 (RFI): now also L1.1
- net at U5.4 (XTA): now also X2.3 (Osc)
- net at AN2.1 (In): now also R12.2
- net at AN1.1 (In): now also R13.2
- new net: C23.2, R13.1
- new net: C20.1, C21.1, L4.2, L5.1
- new net: C21.2, C22.1, C23.1, L5.2
- new net: C13.1, L1.2, R11.1
- new net: C14.1, R11.2
- new net: C14.2, C15.1
- new net: BT1.1 (Inner1), F1.1
- new net: C18.1, C19.2, L2.2, L3.2
- new net: C15.2, R12.1
- new net: C19.1, L4.1
- new net +3.3V: C5.1, C6.1, C7.1, C8.2, C9.1, F1.2, FB1.1, R1.2, R2.2, SW1.2 (B), U1.10 (DVCC), U3.15 (VDDTX), U3.19 (VDDRX), U3.20 (VDDPLL), U3.25 (VDDOSC), U3.28 (VDD), U4.20 (VBAT), U4.23 (VDDIO), U5.1 (VBAT1), U5.15 (VBAT2), U6.1 (VBAT1), U6.15 (VBAT2), X1.4 (Vdc), X2.4 (Vdc)
- no-connect marks 11 -> 13
Other:
- removed sheet Ethernet
- removed sheet LoRa
- removed sheet WiFi
- moved on the sheet: AN1, AN2, U4, X1, X2
